File: mega128board.sch (EAGLE design)
At the start: 6 parts, among them CON1 M161X16_NO_SILK, CON2 M161X16_NO_SILK, CON3 M161X16_NO_SILK, CON4 M161X16_NO_SILK, IC1 MEGA128-A

Commit message: ~
Parts:
- added C1, C2, C3: (no value), rcl:C-EUC0805
- added CON5, CON6, CON7, CON8: M161X16_NO_SILK, SparkFun-Connectors:M161X16_NO_SILK
- added ICSP: M05X2SHD, SparkFun-Connectors:M05X2SHD
- added JP3: M02PTH, SparkFun-Connectors:M02PTH
- added JP4: (no value), jumper:JP2QE
- added LED1: (no value), SparkFun-LED:LED1206
- added R1, R2: (no value), rcl:R-EU_M0805
- added S1: DTSM-6, switch-tact:DTSM-6
Connections:
- new net N$1: C1.1, S1.1, S1.2
- new net N$2: R1.1, S1.3, S1.4
- new net N$3: LED1.C, R2.2
- new net N$5: C3.1, JP3.2, JP4-2.1
- new net N$6: C2.1, JP3.1, JP4-1.1
- net +5V: now also CON6.5, CON7.4, ICSP.2, LED1.A, R1.2
- net AGND: now also CON7.15
- net ALE: now also CON8.11
- net AREF: now also CON7.14
- net AVCC: now also CON7.16
- net GND: now also C1.2, C2.2, C3.2, CON6.6, CON7.5, ICSP.10, ICSP.4, ICSP.6, ICSP.8, R2.1
- net PA0: now also CON7.3
- net PA1: now also CON7.2
- net PA2: now also CON7.1
- net PA3: now also CON8.16
- net PA4: now also CON8.15
- net PA5: now also CON8.14
- net PA6: now also CON8.13
- net PA7: now also CON8.12
- net PB0: now also CON5.10
- net PB1: now also CON5.11, ICSP.7
- net PB2: now also CON5.12
- net PB3: now also CON5.13
- net PB4: now also CON5.14
- net PB5: now also CON5.15
- net PB6: now also CON5.16
- net PB7: now also CON6.1
- net PC0: now also CON8.3
- net PC1: now also CON8.4
- net PC2: now also CON8.5
- net PC3: now also CON8.6
- net PC4: now also CON8.7
- net PC5: now also CON8.8
- net PC6: now also CON8.9
- net PC7: now also CON8.10
- net PD0: now also CON6.9
- net PD1: now also CON6.10
- net PD2: now also CON6.11
- net PD3: now also CON6.12
- net PD4: now also CON6.13
- net PD5: now also CON6.14
- net PD6: now also CON6.15
- net PD7: now also CON6.16
- net PE0: now also CON5.2, ICSP.1
- net PE1: now also CON5.3, ICSP.9
- net PE2: now also CON5.4
- net PE3: now also CON5.5
- net PE4: now also CON5.6
- net PE5: now also CON5.7
- net PE6: now also CON5.8
- net PE7: now also CON5.9
- net PEN: now also CON5.1
- net PF0: now also CON7.13
- net PF1: now also CON7.12
- net PF2: now also CON7.11
- net PF3: now also CON7.10
- net RD: now also CON8.2
- net RESET: now also CON6.4, ICSP.5
- net TCK: now also CON7.9
- net TDI: now also CON7.6
- net TDO: now also CON7.7
- net TMS: now also CON7.8
- net TOSC1: now also CON6.3
- net TOSC2: now also CON6.2
- net WR: now also CON8.1
- net XTAL1: now also CON6.8, JP4-1.2
- net XTAL2: now also CON6.7, JP4-2.2
Other:
- moved on the sheet: CON1, CON2, CON3, CON4
