File: 128.brd (EAGLE design)
At the start: 119.4 x 65.7 mm, 26 parts, among them IC1 MEGA128-A, J1 JTAG, J11 M16PTH, J12 M16PTH, J2 ICSP, J21 M16PTH, J22 M16PTH, J31 M16PTH, J32 M16PTH, J41 M16PTH, J42 M16PTH

Commit message: ~
Parts:
- added U$1: M10X2NOSILK, SparkFun-Connectors:2X10_NOSILK
- JP17: value (none) -> AGND
- JP18: value (none) -> AVCC
- JP3: value M02LOCK -> FQ
- moved C2 123.1 mm to (87.9, 5.46), turned to 270 degrees
- moved JP3 121.7 mm to (87.2, 14.4), turned to 180 degrees
- moved JP17 117.9 mm to (11.8, 68.2), turned to 270 degrees
- moved C1 116.3 mm to (84.5, 5.46), turned to 270 degrees
- moved J1 116.0 mm to (86.5, 76.3), turned to 270 degrees
- moved JP18 103.9 mm to (16.4, 68.3), turned to 270 degrees
- moved JP6 99.7 mm to (77.2, 11.7)
- moved JP5 85.6 mm to (77.3, 7.11)
- moved R2 84.6 mm to (11.7, 17.1), turned to 90 degrees
- moved C5 83.8 mm to (19.3, 14.7), turned to 180 degrees
- moved J2 78.9 mm to (14.1, 77.1), turned to 270 degrees
- moved J11 52.3 mm to (6.35, 59.7)
- moved R12 45.1 mm to (19.3, 10.9)
- moved J12 43.8 mm to (8.89, 59.7)
- moved LED1 39.7 mm to (14.7, 13.2), turned to 90 degrees
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Connections:
- new net +5V1: JP18.1
- new net AGND1: JP17.2
- new net AVCC1: JP18.2
- new net GND1: JP17.1
- new net PB15: J2.7
- new net PE15: J2.9
- new net RESET1: J1.6
- new net RESET23: C11.1, R11.1, S1.1
- new net RESET5: J2.5
- new net TCK1: J1.1
- new net TDI1: J1.9
- new net TDO1: J1.3
- new net TMS1: J1.5
- new net XTAL13: JP5.1
- net +5V: now also J41.4, J42.4; no longer J41.16, J42.16, JP18.1
- net AGND: now also J41.15, J42.15; no longer J41.5, J42.5, JP17.2
- net AVCC: now also J41.16, J42.16; no longer J41.4, J42.4, JP18.2
- net GND: now also J41.5, J42.5; no longer J41.15, J41.6, J42.15, J42.6, JP17.1
- net PA3: now also J31.16, J32.16
- net PA4: now also IC1.47
- net PA5: no longer J31.16, J32.16
- net PB1: no longer J2.7
- net PE1: no longer J2.9
- net RESET: no longer C11.1, J1.6, J2.5, R11.1, S1.1
- net TCK: no longer J1.1
- net TDI: now also J41.6, J42.6; no longer J1.9, J41.7, J42.7
- net TDO: now also J41.7, J42.7; no longer J1.3, J41.8, J42.8
- net TMS: now also J41.8, J42.8; no longer J1.5
- net XTAL1: no longer JP5.1
Routing:
- net GND: track 0.00 -> 289.3 mm, vias 0 -> 4
- net +5V: track 0.00 -> 240.9 mm, vias 0 -> 3
- net PEN: track 0.00 -> 82.1 mm, vias 0 -> 1
- net XTAL1: track 0.00 -> 67.3 mm, vias 0 -> 1
- net PE0: track 0.00 -> 65.6 mm, vias 0 -> 1
- net PB6: track 0.00 -> 40.9 mm, vias 0 -> 1
- net WR: track 0.00 -> 40.6 mm, vias 0 -> 1
- net PB5: track 0.00 -> 40.2 mm, vias 0 -> 1
- net RD: track 0.00 -> 39.9 mm, vias 0 -> 1
- net PB4: track 0.00 -> 39.4 mm, vias 0 -> 1
- net PC0: track 0.00 -> 39.2 mm, vias 0 -> 1
- net PB3: track 0.00 -> 38.7 mm, vias 0 -> 1
- net PA3: track 0.00 -> 38.5 mm, vias 0 -> 1
- net PC1: track 0.00 -> 38.5 mm, vias 0 -> 1
- net PB2: track 0.00 -> 38.0 mm, vias 0 -> 1
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Other:
- board size 119.4 x 65.7 mm -> 117.3 x 86.8 mm

Commit message: ~
Parts:
- removed U$1: M10X2NOSILK, SparkFun-Connectors:2X10_NOSILK
- moved JP17 12.0 mm to (22.9, 63.5), turned to 0 degrees
- moved JP18 6.48 mm to (22.9, 68.6), turned to 0 degrees
- moved JP6 2.67 mm to (79.9, 11.7), turned to 180 degrees
- moved JP3 1.71 mm to (85.6, 13.9), turned to 0 degrees
- moved J2 0.89 mm to (13.2, 77.0)
- moved J1 0.70 mm to (86.6, 77.0)
Connections:
- removed net +5V1: JP18.1
- removed net AGND1: JP17.2
- removed net AVCC1: JP18.2
- removed net GND1: JP17.1
- removed net PB15: J2.7
- removed net PE15: J2.9
- removed net RESET1: J1.6
- removed net RESET23: C11.1, R11.1, S1.1
- removed net RESET5: J2.5
- removed net TCK1: J1.1
- removed net TDI1: J1.9
- removed net TDO1: J1.3
- removed net TMS1: J1.5
- removed net XTAL13: JP5.1
- net +5V: now also JP18.1
- net AGND: now also JP17.2
- net AVCC: now also JP18.2
- net GND: now also JP17.1
- net PB1: now also J2.7
- net PE1: now also J2.9
- net RESET: now also C11.1, J1.6, J2.5, R11.1, S1.1
- net TCK: now also J1.1
- net TDI: now also J1.9
- net TDO: now also J1.3
- net TMS: now also J1.5
- net XTAL1: now also JP5.1
Routing:
- net RESET: track 33.2 -> 203.5 mm, vias 1 -> 3
- net PB1: track 37.3 -> 102.0 mm
- net TCK: track 30.0 -> 86.1 mm
- net TMS: track 30.7 -> 78.1 mm
- net TDO: track 31.4 -> 78.8 mm
- net TDI: track 32.2 -> 64.9 mm
- net PE1: track 37.3 -> 65.0 mm
- net +5V: track 240.9 -> 265.4 mm, vias 3 -> 6
- net GND: track 289.3 -> 306.8 mm, vias 4 -> 2
- net RESET23: track 15.3 -> 0.00 mm
- net AGND: track 34.7 -> 48.3 mm
- net AVCC: track 34.8 -> 42.0 mm
- net N$66: track 18.3 -> 22.5 mm
- net N$65: track 19.6 -> 16.3 mm
- net PE0: track 65.6 -> 67.2 mm
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Other:
- board size 117.3 x 86.8 mm -> 96.7 x 87.1 mm
- board text added: "1"
- board text added: "16"
- board text added: "17"
- board text added: "32"
- board text added: "33"
- board text added: "48"
- board text added: "49"
- board text added: "64"
- board text added: "ICSP"
- board text added: "JTAG"

Commit message: ~
Other:
- board text added: "AG"
- board text added: "AV"
- board text added: "Q"
Changed lines of the file:
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@@
 <wire x1="96.627" y1="86.919" x2="-0.0635" y2="87.1095" width="0.4064" layer="20"/>
 <wire x1="-0.0635" y1="87.1095" x2="0" y2="0" width="0.4064" layer="20"/>
-<text x="1.778" y="61.341" size="2.54" layer="1" font="vector" ratio="23">1</text>
-<text x="1.5875" y="16.891" size="2.54" layer="1" font="vector" ratio="23">16</text>
-<text x="23.9395" y="16.002" size="2.54" layer="1" font="vector" ratio="23">17</text>
-<text x="70.866" y="15.875" size="2.54" layer="1" font="vector" ratio="23">32</text>
-<text x="90.424" y="16.51" size="2.54" layer="1" font="vector" ratio="23">33</text>
-<text x="90.17" y="62.5475" size="2.54" layer="1" font="vector" ratio="23">48</text>
-<text x="72.263" y="79.248" size="2.54" layer="1" font="vector" ratio="23">49</text>
-<text x="26.289" y="83.2485" size="2.54" layer="1" font="vector" ratio="23">64</text>
-<text x="2.413" y="69.977" size="2.54" layer="1" font="vector" ratio="23">ICSP</text>
-<text x="85.979" y="68.2625" size="2.54" layer="1" font="vector" ratio="23">JTAG</text>
+<text x="1.778" y="61.341" size="2.1844" layer="1" font="vector" ratio="16">1</text>
+<text x="1.5875" y="16.891" size="2.1844" layer="1" font="vector" ratio="16">16</text>
+<text x="23.9395" y="16.002" size="2.1844" layer="1" font="vector" ratio="16">17</text>
+<text x="70.866" y="15.875" size="2.1844" layer="1" font="vector" ratio="16">32</text>
+<text x="90.424" y="16.51" size="2.1844" layer="1" font="vector" ratio="16">33</text>
+<text x="90.17" y="62.5475" size="2.1844" layer="1" font="vector" ratio="16">48</text>
+<text x="72.263" y="79.248" size="2.1844" layer="1" font="vector" ratio="16">49</text>
+<text x="26.289" y="83.2485" size="2.1844" layer="1" font="vector" ratio="16">64</text>
+<text x="2.413" y="69.977" size="2.1844" layer="1" font="vector" ratio="16">ICSP</text>
+<text x="85.979" y="68.2625" size="2.1844" layer="1" font="vector" ratio="16">JTAG</text>
+<text x="17.3355" y="69.6595" size="1.778" layer="1" font="vector" ratio="16">AV</text>
+<text x="17.272" y="64.77" size="1.778" layer="1" font="vector" ratio="16">AG</text>
+<text x="91.059" y="11.811" size="1.778" layer="1" font="vector" ratio="16">Q</text>
 </plain>
 <attributes>
@@
 <wire x1="58.57875" y1="65.24625" x2="58.57875" y2="71.02475" width="0.6096" layer="16"/>
 <wire x1="58.57875" y1="71.02475" x2="58.674" y2="71.12" width="0.6096" layer="16"/>
-<wire x1="12.7" y1="5.08" x2="12.7" y2="5.1435" width="0.4064" layer="1"/>
-<wire x1="12.7" y1="5.1435" x2="11.684" y2="6.1595" width="0.4064" layer="1"/>
-<wire x1="11.684" y1="6.1595" x2="11.684" y2="7.0485" width="0.4064" layer="1"/>
-<wire x1="11.684" y1="7.0485" x2="10.922" y2="7.8105" width="0.4064" layer="1"/>
-<wire x1="10.922" y1="7.8105" x2="10.795" y2="7.9375" width="0.4064" layer="1"/>
-<wire x1="10.795" y1="7.9375" x2="8.4455" y2="7.9375" width="0.4064" layer="1"/>
+<wire x1="12.7" y1="7.9375" x2="8.4455" y2="7.9375" width="0.4064" layer="1"/>
 <wire x1="8.4455" y1="7.9375" x2="8.382" y2="8.001" width="0.4064" layer="1"/>
 <wire x1="8.382" y1="8.001" x2="8.3545" y2="8.001" width="0.4064" layer="1"/>
@@
 <wire x1="13.438" y1="14.708" x2="12.7" y2="13.97" width="0.4064" layer="1"/>
 <wire x1="12.7" y1="13.97" x2="12.7" y2="9.5885" width="0.4064" layer="1"/>
-<wire x1="12.7" y1="9.5885" x2="10.922" y2="7.8105" width="0.4064" layer="1"/>
 <wire x1="91.6305" y1="70.612" x2="91.6305" y2="75.6285" width="0.6096" layer="16"/>
+<wire x1="12.7" y1="5.08" x2="12.7" y2="7.9375" width="0.4064" layer="1"/>
+<wire x1="12.7" y1="7.9375" x2="12.7" y2="9.525" width="0.4064" layer="1"/>
+<wire x1="12.7" y1="9.525" x2="12.7" y2="9.5885" width="0" layer="19" extent="1-1"/>
+<wire x1="12.7" y1="7.9375" x2="12.7" y2="9.525" width="0" layer="19" extent="1-16"/>
 </signal>
 <signal name="PA4">

Commit message: ~
Routing:
- added copper zone on layer 1, net N$1
- added copper zone on layer 16, net N$2
- added copper zone on layer 1, net N$3
Changed lines of the file:
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@@
 <param name="mdViaViaSameLayer" value="8mil"/>
 <param name="mnLayersViaInSmd" value="2"/>
-<param name="mdCopperDimension" value="40mil"/>
-<param name="mdDrill" value="40mil"/>
+<param name="mdCopperDimension" value="60mil"/>
+<param name="mdDrill" value="60mil"/>
 <param name="mdSmdStop" value="0mil"/>
 <param name="msWidth" value="10mil"/>
@@
 <wire x1="12.7" y1="7.9375" x2="12.7" y2="9.525" width="0.4064" layer="1"/>
 <wire x1="12.7" y1="9.525" x2="12.7" y2="9.5885" width="0" layer="19" extent="1-1"/>
-<wire x1="12.7" y1="7.9375" x2="12.7" y2="9.525" width="0" layer="19" extent="1-16"/>
 </signal>
 <signal name="PA4">
@@
 <wire x1="21.0185" y1="78.4225" x2="18.288" y2="78.4225" width="0.6096" layer="16"/>
 </signal>
+<signal name="N$1">
+<polygon width="0.4064" layer="1">
+<vertex x="0.762" y="86.36"/>
+<vertex x="95.885" y="86.36"/>
+<vertex x="95.885" y="0.635"/>
+<vertex x="0.6985" y="0.635"/>
+</polygon>
+</signal>
+<signal name="N$2">
+<polygon width="0.4064" layer="16">
+<vertex x="0.889" y="86.106"/>
+<vertex x="95.8215" y="86.106"/>
+<vertex x="95.8215" y="0.635"/>
+<vertex x="0.635" y="0.635"/>
+<vertex x="0.635" y="5.207"/>
+<vertex x="0.508" y="5.207"/>
+<vertex x="0.508" y="86.1695"/>
+<vertex x="1.524" y="86.1695"/>
+</polygon>
+</signal>
+<signal name="N$3">
+<polygon width="0.4064" layer="1">
+<vertex x="56.769" y="40.767"/>
+<vertex x="69.469" y="40.767"/>
+<vertex x="69.469" y="22.987"/>
+<vertex x="56.769" y="22.987"/>
+</polygon>
+</signal>
 </signals>

Commit message: ~
Connections:
- net PEN renamed N$3
Routing:
- net GND: track 307.0 -> 422.5 mm
- net +5V: track 265.4 -> 346.6 mm, vias 6 -> 5
- net RESET: track 203.5 -> 238.0 mm
- net PB1: track 102.0 -> 94.6 mm
- net PC7: track 34.2 -> 37.0 mm
- net N$6: track 0.00 -> 2.73 mm
- net N$10: track 0.00 -> 2.73 mm
- net TOSC2: track 34.7 -> 37.4 mm
- net TOSC1: track 34.0 -> 36.6 mm
- net N$9: track 0.00 -> 2.67 mm
- net N$8: track 0.00 -> 2.67 mm
- net N$7: track 0.00 -> 2.67 mm
- net N$5: track 0.00 -> 2.67 mm
- net N$4: track 0.00 -> 2.67 mm
- net N$12: track 0.00 -> 2.67 mm
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- removed copper zone on layer 1, net N$1
- removed copper zone on layer 16, net N$2
- removed copper zone on layer 1, net N$3 (its old number)

Commit message: ~
Connections:
- net N$3 renamed PEN
Changed lines of the file:
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@@
 <via x="43.053" y="15.24" extent="1-16" drill="0.6" diameter="1.6764" shape="square"/>
 <wire x1="85.09" y1="5.08" x2="84.455" y2="4.611" width="0.254" layer="1"/>
-<wire x1="87.63" y1="5.08" x2="87.884" y2="4.611" width="0.254" layer="1"/>
 <wire x1="27.1145" y1="2.54" x2="43.1165" y2="2.54" width="0.4064" layer="1"/>
 <wire x1="43.1165" y1="2.54" x2="78.867" y2="2.54" width="0.4064" layer="1"/>
@@
 <wire x1="18.0975" y1="3.2385" x2="18.072" y2="3.2385" width="0.4064" layer="1"/>
 <wire x1="18.072" y1="3.2385" x2="18.0365" y2="3.203" width="0.4064" layer="1"/>
-<wire x1="87.63" y1="5.08" x2="87.63" y2="4.826" width="0.4064" layer="1"/>
 <wire x1="87.63" y1="4.826" x2="87.4395" y2="4.6355" width="0.4064" layer="1"/>
 <wire x1="87.4395" y1="4.6355" x2="84.4795" y2="4.6355" width="0.4064" layer="1"/>
@@
 <wire x1="58.674" y1="80.8355" x2="58.674" y2="78.1685" width="0.6096" layer="1"/>
 <wire x1="43.053" y1="7.62" x2="43.053" y2="5.08" width="0.6096" layer="1"/>
+<wire x1="87.63" y1="4.826" x2="87.884" y2="4.826" width="0.4064" layer="1"/>
+<wire x1="87.884" y1="4.826" x2="87.884" y2="4.611" width="0.4064" layer="1"/>
 </signal>
 <signal name="PA4">
@@
 <contactref element="JP5" pad="2"/>
 <contactref element="C1" pad="1"/>
-<wire x1="83.82" y1="6.35" x2="84.455" y2="6.311" width="0.254" layer="1"/>
 <wire x1="85.4202" y1="13.9065" x2="85.4202" y2="8.6487" width="0.6096" layer="16"/>
 <wire x1="85.4202" y1="8.6487" x2="83.8835" y2="7.112" width="0.6096" layer="16"/>
 <wire x1="83.8835" y1="7.112" x2="79.883" y2="7.112" width="0.6096" layer="16"/>
-<wire x1="83.82" y1="6.35" x2="81.5975" y2="6.35" width="0.4064" layer="1"/>
+<wire x1="84.3915" y1="6.35" x2="81.5975" y2="6.35" width="0.4064" layer="1"/>
 <wire x1="81.5975" y1="6.35" x2="80.8355" y2="7.112" width="0.4064" layer="1"/>
 <wire x1="80.8355" y1="7.112" x2="79.883" y2="7.112" width="0.4064" layer="1"/>
+<wire x1="84.3915" y1="6.35" x2="84.3915" y2="6.311" width="0.4064" layer="1"/>
+<wire x1="84.455" y1="6.311" x2="84.3915" y2="6.311" width="0.4064" layer="1"/>
+<wire x1="84.3915" y1="6.311" x2="84.3915" y2="6.2865" width="0.4064" layer="1"/>
 </signal>
 <signal name="N$66">
@@
 <wire x1="6.2865" y1="57.15" x2="8.9535" y2="57.15" width="0.6096" layer="1"/>
 </signal>
-<signal name="N$3">
-<wire x1="6.4135" y1="59.69" x2="8.9535" y2="59.69" width="0.6096" layer="1"/>
+<signal name="N$4">
+<wire x1="35.814" y1="80.8355" x2="35.814" y2="78.1685" width="0.6096" layer="1"/>
+</signal>
+<signal name="N$5">
+<wire x1="38.354" y1="80.8355" x2="38.354" y2="78.1685" width="0.6096" layer="1"/>
+</signal>
+<signal name="N$6">
+<wire x1="40.894" y1="80.899" x2="40.894" y2="78.1685" width="0.6096" layer="1"/>
+</signal>
+<signal name="N$7">
+<wire x1="43.434" y1="80.8355" x2="43.434" y2="78.1685" width="0.6096" layer="1"/>
+</signal>
+<signal name="N$8">
+<wire x1="48.514" y1="80.8355" x2="48.514" y2="78.1685" width="0.6096" layer="1"/>
+</signal>
+<signal name="N$9">
+<wire x1="51.054" y1="80.8355" x2="51.054" y2="78.1685" width="0.6096" layer="1"/>
+</signal>
+<signal name="N$10">
+<wire x1="56.134" y1="80.899" x2="56.134" y2="78.1685" width="0.6096" layer="1"/>
+</signal>
+<signal name="N$11">
+<wire x1="63.754" y1="80.8355" x2="63.754" y2="78.1685" width="0.6096" layer="1"/>
+</signal>
+<signal name="N$12">
+<wire x1="87.8205" y1="24.13" x2="90.4875" y2="24.13" width="0.6096" layer="1"/>
+</signal>
+<signal name="N$13">
+<wire x1="30.353" y1="5.1435" x2="30.353" y2="7.6835" width="0.6096" layer="1"/>
+</signal>
+<signal name="PEN">
 <contactref element="IC1" pad="1"/>
+<wire x1="6.35" y1="59.69" x2="8.9535" y2="59.69" width="0.6096" layer="1"/>
 <contactref element="J11" pad="1"/>
 <contactref element="J12" pad="1"/>
@@
 <wire x1="6.35" y1="59.69" x2="8.89" y2="59.69" width="0.6096" layer="16"/>
 <wire x1="8.89" y1="59.69" x2="15.24" y2="59.69" width="0.6096" layer="16"/>
-<wire x1="40.7543" y1="49.0855" x2="34.2265" y2="49.0855" width="0.4064" layer="1"/>
 <wire x1="34.2265" y1="49.0855" x2="23.622" y2="59.69" width="0.4064" layer="1"/>
 <wire x1="23.622" y1="59.69" x2="15.24" y2="59.69" width="0.4064" layer="1"/>
 <via x="15.24" y="59.69" extent="1-16" drill="0.6" diameter="1.6764" shape="square"/>
 <wire x1="11.43" y1="17.78" x2="11.7475" y2="17.995" width="0.254" layer="1"/>
-<wire x1="13.7795" y1="59.69" x2="15.24" y2="59.69" width="0.4064" layer="1"/>
+<wire x1="13.7795" y1="59.69" x2="15.24" y2="59.69" width="0.6096" layer="1"/>
 <wire x1="11.7475" y1="17.995" x2="11.7475" y2="57.658" width="0.6096" layer="1"/>
-<wire x1="11.7475" y1="57.658" x2="13.7795" y2="59.69" width="0.4064" layer="1"/>
-<wire x1="6.4135" y1="59.69" x2="6.35" y2="59.69" width="0.6096" layer="1"/>
-</signal>
-<signal name="N$4">
-<wire x1="35.814" y1="80.8355" x2="35.814" y2="78.1685" width="0.6096" layer="1"/>
-</signal>
-<signal name="N$5">
-<wire x1="38.354" y1="80.8355" x2="38.354" y2="78.1685" width="0.6096" layer="1"/>
-</signal>
-<signal name="N$6">
-<wire x1="40.894" y1="80.899" x2="40.894" y2="78.1685" width="0.6096" layer="1"/>
-</signal>
-<signal name="N$7">
-<wire x1="43.434" y1="80.8355" x2="43.434" y2="78.1685" width="0.6096" layer="1"/>
-</signal>
-<signal name="N$8">
-<wire x1="48.514" y1="80.8355" x2="48.514" y2="78.1685" width="0.6096" layer="1"/>
-</signal>
-<signal name="N$9">
-<wire x1="51.054" y1="80.8355" x2="51.054" y2="78.1685" width="0.6096" layer="1"/>
-</signal>
-<signal name="N$10">
-<wire x1="56.134" y1="80.899" x2="56.134" y2="78.1685" width="0.6096" layer="1"/>
-</signal>
-<signal name="N$11">
-<wire x1="63.754" y1="80.8355" x2="63.754" y2="78.1685" width="0.6096" layer="1"/>
-</signal>
-<signal name="N$12">
-<wire x1="87.8205" y1="24.13" x2="90.4875" y2="24.13" width="0.6096" layer="1"/>
-</signal>
-<signal name="N$13">
-<wire x1="30.353" y1="5.1435" x2="30.353" y2="7.6835" width="0.6096" layer="1"/>
+<wire x1="11.7475" y1="57.658" x2="13.7795" y2="59.69" width="0.6096" layer="1"/>
+<wire x1="34.2265" y1="49.0855" x2="40.7543" y2="49.0855" width="0.4064" layer="1"/>
 </signal>
 </signals>
-<errors>
-</errors>
 </board>
 </drawing>
