File: 128.sch (EAGLE design)
At the start: 21 parts, among them CON1 M161X16_NO_SILK, CON2 M161X16_NO_SILK, CON3 M161X16_NO_SILK, CON4 M161X16_NO_SILK, CON5 M161X16_NO_SILK, CON6 M161X16_NO_SILK, CON7 M161X16_NO_SILK, CON8 M161X16_NO_SILK, IC1 MEGA128-A

Commit message: ~
Parts:
- removed C3: (no value), rcl:C-EUC0805
- removed CON1, CON2, CON3, CON4, CON5, CON6, CON7, CON8: M161X16_NO_SILK, SparkFun-Connectors:M161X16_NO_SILK
- removed ICSP, JTAG: M05X2SHD, SparkFun-Connectors:M05X2SHD
- removed JP1: M02PTH, SparkFun-Connectors:M02PTH
- removed JP2: (no value), jumper:JP2QE
- removed R1: (no value), rcl:R-EU_M0805
- added C11: 0.1mkF, resistor:C-EUC0805
- added C5: 100nF, resistor:C-EUC0805
- added J1: JTAG, SparkFun-Connectors:M05X2SHD_LOCK
- added J11, J12, J21, J22, J31, J32, J41, J42: M16PTH, SparkFun-Connectors:M16PTH
- added J2: ICSP, SparkFun-Connectors:M05X2SHD_LOCK
- added JP17, JP18, JP5, JP6: (no value), SparkFun-Passives:JUMPER-2PTH
- added JP4: USBSMD, SparkFun-Connectors:USBSMD
- added R11: 10K, resistor:R-EU_R0805
- added R12: 600, resistor:R-EU_R0805
- C1, C2: value (none) -> 22pF; device rcl:C-EUC0805 -> resistor:C-EUC0805
- JP3: value M02PTH -> M02LOCK; device SparkFun-Connectors:M02PTH -> SparkFun-Connectors:M02LOCK
- R2: value (none) -> 1K; device rcl:R-EU_M0805 -> resistor:R-EU_R0805
- S1: value DTSM-6 -> reset; device switch-tact:DTSM-6 -> SparkFun-Electromechanical:SWITCH-MOMENTARY-2SMD-2
Connections:
- removed net N$1: C1.1, S1.1, S1.2
- removed net N$2: R1.1, S1.3, S1.4
- removed net N$3: LED1.C, R2.2
- removed net N$5: C3.1, JP1.2, JP2-2.2
- removed net N$6: C2.1, JP1.1, JP2-1.2
- removed net N$7: JP2-2.1
- new net N$65: C1.1, JP3.1, JP5.2
- new net N$66: C2.1, JP3.2, JP6.1
- new net N$67: LED1.A, R12.1
- net +5V: now also C5.1, J1.4, J1.7, J2.2, J21.5, J22.5, J41.16, J42.16, JP18.1, JP4.VBUS, R11.2, R12.2, R2.1; no longer CON2.5, CON4.4, CON6.5, CON7.4, ICSP.2, JTAG.4, JTAG.7, LED1.A, R1.2
- net AGND: now also J41.5, J42.5, JP17.2; no longer CON4.15, CON7.15
- net ALE: now also J31.11, J32.11; no longer CON3.11, CON8.11
- net AREF: now also J41.14, J42.14; no longer CON4.14, CON7.14
- net AVCC: now also J41.4, J42.4, JP18.2; no longer CON4.16, CON7.16
- net GND: now also C11.2, C5.2, J1.10, J1.2, J2.10, J2.4, J2.6, J2.8, J21.6, J22.6, J41.15, J41.6, J42.15, J42.6, JP17.1, JP4.GND, LED1.C, S1.1; no longer C3.2, CON2.6, CON4.5, CON6.6, CON7.5, ICSP.10, ICSP.4, ICSP.6, ICSP.8, JTAG.10, JTAG.2, R2.1
- net PA0: now also J41.3, J42.3; no longer CON4.3, CON7.3
- net PA1: now also J41.2, J42.2; no longer CON4.2, CON7.2
- net PA2: now also J41.1, J42.1; no longer CON4.1, CON7.1
- net PA3: no longer CON3.16, CON8.16
- net PA4: now also J31.15, J32.15; no longer CON3.15, CON8.15, IC1.(AD4)PA4
- net PA5: now also J31.14, J31.16, J32.14, J32.16; no longer CON3.14, CON8.14
- net PA6: now also J31.13, J32.13; no longer CON3.13, CON8.13
- net PA7: now also J31.12, J32.12; no longer CON3.12, CON8.12
- net PB0: now also J11.10, J12.10; no longer CON1.10, CON5.10
- net PB1: now also J11.11, J12.11, J2.7; no longer CON1.11, CON5.11, ICSP.7
- net PB2: now also J11.12, J12.12; no longer CON1.12, CON5.12
- net PB3: now also J11.13, J12.13; no longer CON1.13, CON5.13
- net PB4: now also J11.14, J12.14; no longer CON1.14, CON5.14
- net PB5: now also J11.15, J12.15; no longer CON1.15, CON5.15
- net PB6: now also J11.16, J12.16; no longer CON1.16, CON5.16
- net PB7: now also J21.1, J22.1; no longer CON2.1, CON6.1
- net PC0: now also J31.3, J32.3; no longer CON3.3, CON8.3
- net PC1: now also J31.4, J32.4; no longer CON3.4, CON8.4
- net PC2: now also J31.5, J32.5; no longer CON3.5, CON8.5
- net PC3: now also J31.6, J32.6; no longer CON3.6, CON8.6
- net PC4: now also J31.7, J32.7; no longer CON3.7, CON8.7
- net PC5: now also J31.8, J32.8; no longer CON3.8, CON8.8
- net PC6: now also J31.9, J32.9; no longer CON3.9, CON8.9
- net PC7: now also J31.10, J32.10; no longer CON3.10, CON8.10
- net PD0: now also J21.9, J22.9; no longer CON2.9, CON6.9
- net PD1: now also J21.10, J22.10; no longer CON2.10, CON6.10
- net PD2: now also J21.11, J22.11; no longer CON2.11, CON6.11
- net PD3: now also J21.12, J22.12; no longer CON2.12, CON6.12
- net PD4: now also J21.13, J22.13; no longer CON2.13, CON6.13
- net PD5: now also J21.14, J22.14; no longer CON2.14, CON6.14
- net PD6: now also J21.15, J22.15; no longer CON2.15, CON6.15
- net PD7: now also J21.16, J22.16; no longer CON2.16, CON6.16
- net PE0: now also J11.2, J12.2, J2.1; no longer CON1.2, CON5.2, ICSP.1
- net PE1: now also J11.3, J12.3, J2.9; no longer CON1.3, CON5.3, ICSP.9
- net PE2: now also J11.4, J12.4; no longer CON1.4, CON5.4
- net PE3: now also J11.5, J12.5; no longer CON1.5, CON5.5
- net PE4: now also J11.6, J12.6; no longer CON1.6, CON5.6
- net PE5: now also J11.7, J12.7; no longer CON1.7, CON5.7
- net PE6: now also J11.8, J12.8; no longer CON1.8, CON5.8
- net PE7: now also J11.9, J12.9; no longer CON1.9, CON5.9
- net PEN: now also J11.1, J12.1, R2.2; no longer CON1.1, CON5.1
- net PF0: now also J41.13, J42.13; no longer CON4.13, CON7.13
- net PF1: now also J41.12, J42.12; no longer CON4.12, CON7.12
- net PF2: now also J41.11, J42.11; no longer CON4.11, CON7.11
- net PF3: now also J41.10, J42.10; no longer CON4.10, CON7.10
- net RD: now also J31.2, J32.2; no longer CON3.2, CON8.2
- net RESET: now also C11.1, J1.6, J2.5, J21.4, J22.4, R11.1, S1.2; no longer CON2.4, CON6.4, ICSP.5, JTAG.6
- net TCK: now also J1.1, J41.9, J42.9; no longer CON4.9, CON7.9, JTAG.1
- net TDI: now also J1.9, J41.7, J42.7; no longer CON4.6, CON7.6
- net TDO: now also J1.3, J41.8, J42.8; no longer CON4.7, CON7.7, JTAG.3
- net TMS: now also J1.5; no longer CON4.8, CON7.8, JTAG.5
- net TOSC1: now also J21.3, J22.3; no longer CON2.3, CON6.3
- net TOSC2: now also J21.2, J22.2; no longer CON2.2, CON6.2
- net WR: now also J31.1, J32.1; no longer CON3.1, CON8.1
- net XTAL1: now also J21.8, J22.8, JP5.1, JP6.2; no longer CON2.8, CON6.8, JP2-1.1
- net XTAL2: now also J21.7, J22.7; no longer CON2.7, CON6.7
Other:
- moved on the sheet: C1, C2, IC1, JP3, LED1, R2

Commit message: ~
Parts:
- added U$1: M10X2NOSILK, SparkFun-Connectors:M10X2NOSILK
- JP17: value (none) -> AGND
- JP18: value (none) -> AVCC
- JP3: value M02LOCK -> FQ
Connections:
- new net +5V1: JP18.1
- new net AGND1: JP17.2
- new net AVCC1: JP18.2
- new net GND1: JP17.1
- new net PB15: J2.7
- new net PE15: J2.9
- new net RESET1: J1.6
- new net RESET23: C11.1, R11.1, S1.2
- new net RESET5: J2.5
- new net TCK1: J1.1
- new net TDI1: J1.9
- new net TDO1: J1.3
- new net TMS1: J1.5
- new net XTAL13: JP5.1
- net +5V: now also J41.4, J42.4; no longer J41.16, J42.16, JP18.1
- net AGND: now also J41.15, J42.15; no longer J41.5, J42.5, JP17.2
- net AVCC: now also J41.16, J42.16; no longer J41.4, J42.4, JP18.2
- net GND: now also J41.5, J42.5; no longer J41.15, J41.6, J42.15, J42.6, JP17.1
- net PA3: now also J31.16, J32.16
- net PA4: now also IC1.(AD4)PA4
- net PA5: no longer J31.16, J32.16
- net PB1: no longer J2.7
- net PE1: no longer J2.9
- net RESET: no longer C11.1, J1.6, J2.5, R11.1, S1.2
- net TCK: no longer J1.1
- net TDI: now also J41.6, J42.6; no longer J1.9, J41.7, J42.7
- net TDO: now also J41.7, J42.7; no longer J1.3, J41.8, J42.8
- net TMS: now also J41.8, J42.8; no longer J1.5
- net XTAL1: no longer JP5.1

Commit message: ~
Parts:
- removed U$1: M10X2NOSILK, SparkFun-Connectors:M10X2NOSILK
Connections:
- removed net +5V1: JP18.1
- removed net AGND1: JP17.2
- removed net AVCC1: JP18.2
- removed net GND1: JP17.1
- removed net PB15: J2.7
- removed net PE15: J2.9
- removed net RESET1: J1.6
- removed net RESET23: C11.1, R11.1, S1.2
- removed net RESET5: J2.5
- removed net TCK1: J1.1
- removed net TDI1: J1.9
- removed net TDO1: J1.3
- removed net TMS1: J1.5
- removed net XTAL13: JP5.1
- net +5V: now also JP18.1
- net AGND: now also JP17.2
- net AVCC: now also JP18.2
- net GND: now also JP17.1
- net PB1: now also J2.7
- net PE1: now also J2.9
- net RESET: now also C11.1, J1.6, J2.5, R11.1, S1.2
- net TCK: now also J1.1
- net TDI: now also J1.9
- net TDO: now also J1.3
- net TMS: now also J1.5
- net XTAL1: now also JP5.1
Changed lines of the file:
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@@
 <part name="GND6" library="supply1" deviceset="GND" device=""/>
 <part name="P+7" library="supply1" deviceset="+5V" device=""/>
-<part name="U$1" library="SparkFun-Connectors" deviceset="M10X2" device="NOSILK"/>
 </parts>
 <sheets>
@@
 <instance part="GND6" gate="1" x="-58.42" y="73.66"/>
 <instance part="P+7" gate="1" x="-66.04" y="81.28" rot="R270"/>
-<instance part="U$1" gate="G$1" x="-53.34" y="0"/>
 </instances>
 <busses>
@@
 <label x="129.54" y="81.28" size="1.778" layer="95"/>
 </segment>
+<segment>
+<pinref part="JP17" gate="A" pin="1"/>
+<wire x1="27.94" y1="124.46" x2="15.24" y2="124.46" width="0.1524" layer="91"/>
+<label x="15.24" y="124.46" size="1.778" layer="95"/>
+<junction x="27.94" y="124.46"/>
+</segment>
 </net>
 <net name="+5V" class="0">
@@
 <junction x="152.4" y="83.82"/>
 </segment>
+<segment>
+<pinref part="JP18" gate="A" pin="1"/>
+<wire x1="27.94" y1="111.76" x2="15.24" y2="111.76" width="0.1524" layer="91"/>
+<label x="15.24" y="111.76" size="1.778" layer="95"/>
+<junction x="27.94" y="111.76"/>
+</segment>
 </net>
 <net name="N$67" class="0">
@@
 <junction x="5.08" y="27.94"/>
 </segment>
+<segment>
+<pinref part="S1" gate="G$1" pin="2"/>
+<wire x1="-48.26" y1="109.22" x2="-40.64" y2="109.22" width="0.1524" layer="91"/>
+<pinref part="R11" gate="G$1" pin="1"/>
+<wire x1="-40.64" y1="109.22" x2="-40.64" y2="111.76" width="0.1524" layer="91"/>
+<pinref part="C11" gate="G$1" pin="1"/>
+<wire x1="-40.64" y1="109.22" x2="-40.64" y2="106.68" width="0.1524" layer="91"/>
+<junction x="-40.64" y="109.22"/>
+<junction x="-48.26" y="109.22"/>
+<label x="-55.88" y="109.22" size="1.778" layer="95"/>
+<wire x1="-48.26" y1="109.22" x2="-55.88" y2="109.22" width="0.1524" layer="91"/>
+</segment>
+<segment>
+<pinref part="J2" gate="G$1" pin="5"/>
+<wire x1="-93.98" y1="48.26" x2="-101.6" y2="48.26" width="0.1524" layer="91"/>
+<label x="-101.6" y="48.26" size="1.778" layer="95"/>
+<junction x="-93.98" y="48.26"/>
+</segment>
+<segment>
+<pinref part="J1" gate="G$1" pin="6"/>
+<wire x1="134.62" y1="116.84" x2="144.78" y2="116.84" width="0.1524" layer="91"/>
+<label x="142.24" y="116.84" size="1.778" layer="95"/>
+<junction x="134.62" y="116.84"/>
+</segment>
 </net>
 <net name="XTAL2" class="0">
@@
 <label x="-66.04" y="114.3" size="1.778" layer="95"/>
 </segment>
+<segment>
+<pinref part="JP5" gate="A" pin="1"/>
+<wire x1="-96.52" y1="114.3" x2="-101.6" y2="114.3" width="0.1524" layer="91"/>
+</segment>
 </net>
 <net name="AREF" class="0">
@@
 <junction x="152.4" y="53.34"/>
 </segment>
+<segment>
+<wire x1="43.18" y1="111.76" x2="30.48" y2="111.76" width="0.1524" layer="91"/>
+<pinref part="JP18" gate="A" pin="2"/>
+<label x="40.64" y="111.76" size="1.778" layer="95"/>
+<junction x="30.48" y="111.76"/>
+</segment>
 </net>
 <net name="AGND" class="0">
@@
 <label x="129.54" y="55.88" size="1.778" layer="95"/>
 <junction x="152.4" y="55.88"/>
+</segment>
+<segment>
+<pinref part="JP17" gate="A" pin="2"/>
+<wire x1="30.48" y1="124.46" x2="43.18" y2="124.46" width="0.1524" layer="91"/>
+<label x="40.64" y="124.46" size="1.778" layer="95"/>
+<junction x="30.48" y="124.46"/>
 </segment>
 </net>
@@
 <label x="129.54" y="78.74" size="1.778" layer="95"/>
 </segment>
+<segment>
+<pinref part="J1" gate="G$1" pin="9"/>
+<wire x1="119.38" y1="111.76" x2="104.14" y2="111.76" width="0.1524" layer="91"/>
+<label x="104.14" y="111.76" size="1.778" layer="95"/>
+<junction x="119.38" y="111.76"/>
+</segment>
 </net>
 <net name="TDO" class="0">
@@
 <label x="129.54" y="76.2" size="1.778" layer="95"/>
 </segment>
+<segment>
+<pinref part="J1" gate="G$1" pin="3"/>
+<wire x1="119.38" y1="119.38" x2="104.14" y2="119.38" width="0.1524" layer="91"/>
+<label x="104.14" y="119.38" size="1.778" layer="95"/>
+<junction x="119.38" y="119.38"/>
+</segment>
 </net>
 <net name="TMS" class="0">
@@
 <junction x="152.4" y="73.66"/>
 </segment>
+<segment>
+<pinref part="J1" gate="G$1" pin="5"/>
+<wire x1="119.38" y1="116.84" x2="104.14" y2="116.84" width="0.1524" layer="91"/>
+<label x="104.14" y="116.84" size="1.778" layer="95"/>
+<junction x="119.38" y="116.84"/>
+</segment>
 </net>
 <net name="TCK" class="0">
@@
 <junction x="152.4" y="71.12"/>
 </segment>
+<segment>
+<pinref part="J1" gate="G$1" pin="1"/>
+<wire x1="119.38" y1="121.92" x2="104.14" y2="121.92" width="0.1524" layer="91"/>
+<label x="104.14" y="121.92" size="1.778" layer="95"/>
+<junction x="119.38" y="121.92"/>
+</segment>
 </net>
 <net name="PF3" class="0">
@@
 <junction x="5.08" y="71.12"/>
 </segment>
+<segment>
+<pinref part="J2" gate="G$1" pin="7"/>
+<wire x1="-93.98" y1="45.72" x2="-101.6" y2="45.72" width="0.1524" layer="91"/>
+<label x="-101.6" y="45.72" size="1.778" layer="95"/>
+<junction x="-93.98" y="45.72"/>
+</segment>
 </net>
 <net name="PB0" class="0">
@@
 <junction x="5.08" y="91.44"/>
 </segment>
+<segment>
+<pinref part="J2" gate="G$1" pin="9"/>
+<wire x1="-93.98" y1="43.18" x2="-101.6" y2="43.18" width="0.1524" layer="91"/>
+<label x="-101.6" y="43.18" size="1.778" layer="95"/>
+<junction x="-93.98" y="43.18"/>
+</segment>
 </net>
 <net name="PE0" class="0">
@@
 </segment>
 </net>
-<net name="AGND1" class="0">
-<segment>
-<pinref part="JP17" gate="A" pin="2"/>
-<wire x1="30.48" y1="124.46" x2="43.18" y2="124.46" width="0.1524" layer="91"/>
-<label x="40.64" y="124.46" size="1.778" layer="95"/>
-<junction x="30.48" y="124.46"/>
-</segment>
-</net>
-<net name="AVCC1" class="0">
-<segment>
-<wire x1="43.18" y1="111.76" x2="30.48" y2="111.76" width="0.1524" layer="91"/>
-<pinref part="JP18" gate="A" pin="2"/>
-<label x="40.64" y="111.76" size="1.778" layer="95"/>
-<junction x="30.48" y="111.76"/>
-</segment>
-</net>
-<net name="+5V1" class="0">
-<segment>
-<pinref part="JP18" gate="A" pin="1"/>
-<wire x1="27.94" y1="111.76" x2="15.24" y2="111.76" width="0.1524" layer="91"/>
-<label x="15.24" y="111.76" size="1.778" layer="95"/>
-<junction x="27.94" y="111.76"/>
-</segment>
-</net>
-<net name="GND1" class="0">
-<segment>
-<pinref part="JP17" gate="A" pin="1"/>
-<wire x1="27.94" y1="124.46" x2="15.24" y2="124.46" width="0.1524" layer="91"/>
-<label x="15.24" y="124.46" size="1.778" layer="95"/>
-<junction x="27.94" y="124.46"/>
-</segment>
-</net>
-<net name="RESET1" class="0">
-<segment>
-<pinref part="J1" gate="G$1" pin="6"/>
-<wire x1="134.62" y1="116.84" x2="144.78" y2="116.84" width="0.1524" layer="91"/>
-<label x="142.24" y="116.84" size="1.778" layer="95"/>
-<junction x="134.62" y="116.84"/>
-</segment>
-</net>
-<net name="TDI1" class="0">
-<segment>
-<pinref part="J1" gate="G$1" pin="9"/>
-<wire x1="119.38" y1="111.76" x2="104.14" y2="111.76" width="0.1524" layer="91"/>
-<label x="104.14" y="111.76" size="1.778" layer="95"/>
-<junction x="119.38" y="111.76"/>
-</segment>
-</net>
-<net name="TDO1" class="0">
-<segment>
-<pinref part="J1" gate="G$1" pin="3"/>
-<wire x1="119.38" y1="119.38" x2="104.14" y2="119.38" width="0.1524" layer="91"/>
-<label x="104.14" y="119.38" size="1.778" layer="95"/>
-<junction x="119.38" y="119.38"/>
-</segment>
-</net>
-<net name="TMS1" class="0">
-<segment>
-<pinref part="J1" gate="G$1" pin="5"/>
-<wire x1="119.38" y1="116.84" x2="104.14" y2="116.84" width="0.1524" layer="91"/>
-<label x="104.14" y="116.84" size="1.778" layer="95"/>
-<junction x="119.38" y="116.84"/>
-</segment>
-</net>
-<net name="TCK1" class="0">
-<segment>
-<pinref part="J1" gate="G$1" pin="1"/>
-<wire x1="119.38" y1="121.92" x2="104.14" y2="121.92" width="0.1524" layer="91"/>
-<label x="104.14" y="121.92" size="1.778" layer="95"/>
-<junction x="119.38" y="121.92"/>
-</segment>
-</net>
-<net name="RESET23" class="0">
-<segment>
-<pinref part="S1" gate="G$1" pin="2"/>
-<wire x1="-48.26" y1="109.22" x2="-40.64" y2="109.22" width="0.1524" layer="91"/>
-<pinref part="R11" gate="G$1" pin="1"/>
-<wire x1="-40.64" y1="109.22" x2="-40.64" y2="111.76" width="0.1524" layer="91"/>
-<pinref part="C11" gate="G$1" pin="1"/>
-<wire x1="-40.64" y1="109.22" x2="-40.64" y2="106.68" width="0.1524" layer="91"/>
-<junction x="-40.64" y="109.22"/>
-<junction x="-48.26" y="109.22"/>
-<label x="-55.88" y="109.22" size="1.778" layer="95"/>
-<wire x1="-48.26" y1="109.22" x2="-55.88" y2="109.22" width="0.1524" layer="91"/>
-</segment>
-</net>
-<net name="XTAL13" class="0">
-<segment>
-<pinref part="JP5" gate="A" pin="1"/>
-<wire x1="-96.52" y1="114.3" x2="-101.6" y2="114.3" width="0.1524" layer="91"/>
-</segment>
-</net>
-<net name="RESET5" class="0">
-<segment>
-<pinref part="J2" gate="G$1" pin="5"/>
-<wire x1="-93.98" y1="48.26" x2="-101.6" y2="48.26" width="0.1524" layer="91"/>
-<label x="-101.6" y="48.26" size="1.778" layer="95"/>
-<junction x="-93.98" y="48.26"/>
-</segment>
-</net>
-<net name="PB15" class="0">
-<segment>
-<pinref part="J2" gate="G$1" pin="7"/>
-<wire x1="-93.98" y1="45.72" x2="-101.6" y2="45.72" width="0.1524" layer="91"/>
-<label x="-101.6" y="45.72" size="1.778" layer="95"/>
-<junction x="-93.98" y="45.72"/>
-</segment>
-</net>
-<net name="PE15" class="0">
-<segment>
-<pinref part="J2" gate="G$1" pin="9"/>
-<wire x1="-93.98" y1="43.18" x2="-101.6" y2="43.18" width="0.1524" layer="91"/>
-<label x="-101.6" y="43.18" size="1.778" layer="95"/>
-<junction x="-93.98" y="43.18"/>
-</segment>
-</net>

Commit message: ~
Connections:
- net PEN renamed N$3
Changed lines of the file:
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@@
 </segment>
 </net>
-<net name="PEN" class="0">
+<net name="N$3" class="0">
 <segment>
 <pinref part="IC1" gate="G$1" pin="PEN"/>

Commit message: ~
Connections:
- net N$3 renamed PEN
